File: Schematics/JoyStick.kicad_pcb (KiCad board)
At the start: 4 copper layers, 74.6 x 61.1 mm, 98 parts, among them J1 Conn_01x06, J2 Conn_01x07, J3 Conn_01x02, J4 Conn_01x06, J5 Conn_01x02, J6 Conn_01x05, J7 Conn_01x02, M1 Motor_DC, M2 Motor_DC, Q1 NPN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

Commit message: fix for motor pull down
fix for
Connections:
- R21 pad 1: 5V -> GND
- R32 pad 1: 5V_2 -> GND
Routing:
- net 5V: track 33.9 -> 32.4 mm, vias 12 -> 11
- net 5V_2: track 19.0 -> 17.8 mm, vias 10 -> 9
- net GND: vias 25 -> 27
